File: CM5_MINIMA_REV3-main/CM5_MINIMA_3.kicad_pcb (KiCad board)
At the start: 6 copper layers, 61.4 x 83.1 mm, 117 parts, among them CN1 SM02B-SRSS-TB (LF)(SN), J1 GLPLX-SMT-188S7, J101 TYPEC-305-ACP16H458, J2 Conn_01x04_Pin, J501 GT-HD001B-CNNG1, J502 I2C, J503 SPI, J601 JST_SHBM04B-SRSS-TB, J701 Bus_M.2_Socket_M, J802 Conn_01x22_Female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

Commit message: update
Routing:
- net /CM5/MISO_GPIO19: track 45.0 -> 64.3 mm, vias 2 -> 3
- net /CM5/ETH_nLED_ACTIVITY: track 31.3 -> 36.8 mm, vias 2 -> 3
- net /CM5/IRQ_GPIO26: track 49.3 -> 51.8 mm, vias 2 -> 3
- net /CM5/SCLK_GPIO21: track 64.2 -> 65.3 mm
- net +3V3_PI: track 192.1 -> 191.0 mm, vias 14 -> 13
- net /CM5/MOSI_GPIO20: track 52.4 -> 52.9 mm
- net GND: vias 377 -> 376
