File: CM5_MINIMA_REV3-main/zigbee.kicad_sch (KiCad schematic)
At the start: 4 parts, among them J2 Conn_01x04_Pin, U2 MGM240LD22VIF2

Commit message: Revert CM5_MINIMA_REV3-main to pre-warning-fix state (feae2c2) - fix component mismatches
Parts:
- U2: footprint CM5_MINIMA_local:MGM240L_SIL -> Zigbee MGM240LD22VIF2:MGM240L_SIL
Changed lines of the file:
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@@
 			)
 		)
-		(property "Footprint" "CM5_MINIMA_local:MGM240L_SIL"
+		(property "Footprint" "Zigbee MGM240LD22VIF2:MGM240L_SIL"
 			(at 113.03 83.82 0)
 			(effects

Commit message: warning fix - 17 left
Parts:
- U2: footprint Zigbee MGM240LD22VIF2:MGM240L_SIL -> CM5_MINIMA_local:MGM240L_SIL
Changed lines of the file:
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@@
 			)
 		)
-		(property "Footprint" "Zigbee MGM240LD22VIF2:MGM240L_SIL"
+		(property "Footprint" "CM5_MINIMA_local:MGM240L_SIL"
 			(at 113.03 83.82 0)
 			(effects
