File: CM5_MINIMA_REV3-main/CM5.kicad_sch (KiCad schematic)
At the start: 5 parts, among them CN1 SM02B-SRSS-TB (LF)(SN), M303 Compute-Module-4_H1.5mm

Commit message: Revert CM5_MINIMA_REV3-main to pre-warning-fix state (feae2c2) - fix component mismatches
Parts:
- CN1: footprint Connector_JST:JST_SH_SM02B-SRSS-TB_1x02-1MP_P1.00mm_Horizontal -> EasyEDA:CONN-SMD_2P-P1.00_SM02B-SRSS-TB-LF-SN; symbol Connector_Generic:Conn_01x02 -> EasyEDA:SM02B-SRSS-TB(LF)(SN)
- M303: footprint CM5_MINIMA_local:Compute-Module-4_H1.5mm -> Antmicro-footprints:Compute-Module-4_H1.5mm
- Module301: footprint CM5_MINIMA_local:Raspberry-Pi-5-Compute-Module_GPIO -> CM5IO:Raspberry-Pi-5-Compute-Module_GPIO; symbol CM5_IO:ComputeModule5-CM5_GPIO -> New_Library:ComputeModule5-CM5_GPIO
- Module302: footprint CM5_MINIMA_local:Raspberry-Pi-5-Compute-Module_HSS -> CM5IO:Raspberry-Pi-5-Compute-Module_HSS; symbol CM5_IO:ComputeModule5-CM5_HSS -> New_Library:ComputeModule5-CM5_HSS
Connections:
- net +BATT: now also CN1.1; no longer CN1.2 (Pin_2)
- net GND: now also CN1.2; no longer CN1.1 (Pin_1), M303.1
- no-connect marks 63 -> 65
Changed lines of the file:
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@@
 	)
 	(no_connect
+		(at 123.19 245.11)
+	)
+	(no_connect
 		(at 86.36 165.1)
 	)
@@
 	)
 	(no_connect
+		(at 123.19 232.41)
+	)
+	(no_connect
 		(at 161.29 172.72)
 	)
@@
 	)
 	(symbol
-		(lib_id "power:GND")
-		(at 356.87 247.65 0)
-		(unit 1)
-		(exclude_from_sim no)
-		(in_bom yes)
-		(on_board yes)
-		(dnp no)
-		(property "Reference" "#PWR011"
-			(at 356.87 254 0)
-			(effects
-				(font
-					(size 1.27 1.27)
-				)
-				(hide yes)
-			)
-		)
-		(property "Value" "GND"
-			(at 356.997 252.0442 0)
-			(effects
-				(font
-					(size 1.27 1.27)
-				)
-			)
-		)
-		(property "Footprint" ""
-			(at 356.87 247.65 0)
-			(effects
-				(font
-					(size 1.27 1.27)
-				)
-				(hide yes)
-			)
-		)
-		(property "Datasheet" ""
-			(at 356.87 247.65 0)
-			(effects
-				(font
-					(size 1.27 1.27)
-				)
-				(hide yes)
-			)
-		)
-		(property "Description" "Power symbol creates a global label with name \"GND\" , ground"
-			(at 356.87 247.65 0)
-			(effects
-				(font
-					(size 1.27 1.27)
-				)
-				(hide yes)
-			)
-		)
-		(pin "1"
-		)
-		(instances
-			(project "CM5_MINIMA_3"
-				(path "/b33e81d6-18a9-4b9d-a239-76a7c253462f/45540f0b-d892-4f71-86ad-b9f245bcefda"
-					(reference "#PWR011")
-					(unit 1)
-				)
-			)
-		)
-	)
-	(symbol
-		(lib_id "CM5_IO:ComputeModule5-CM5_HSS")
+		(lib_id "New_Library:ComputeModule5-CM5_HSS")
 		(at 298.45 135.89 0)
 		(unit 1)
@@
 			)
 		)
-		(property "Footprint" "CM5_MINIMA_local:Raspberry-Pi-5-Compute-Module_HSS"
+		(property "Footprint" "CM5IO:Raspberry-Pi-5-Compute-Module_HSS"
 			(at 300.99 136.144 0)
 			(effects
@@
 	)
 	(symbol
-		(lib_id "Connector_Generic:Conn_01x02")
-		(at 118.11 240.03 180)
+		(lib_id "EasyEDA:SM02B-SRSS-TB(LF)(SN)")
+		(at 119.38 238.76 270)
 		(unit 1)
 		(exclude_from_sim no)
@@
 		(fields_autoplaced yes)
 		(property "Reference" "CN1"
-			(at 118.11 231.14 0)
+			(at 118.11 224.79 90)
 			(effects
 				(font
@@
 		)
 		(property "Value" "SM02B-SRSS-TB (LF)(SN)"
-			(at 118.11 233.68 0)
+			(at 118.11 227.33 90)
 			(effects
 				(font
@@
 			)
 		)
-		(property "Footprint" "Connector_JST:JST_SH_SM02B-SRSS-TB_1x02-1MP_P1.00mm_Horizontal"
-			(at 118.11 240.03 0)
+		(property "Footprint" "EasyEDA:CONN-SMD_2P-P1.00_SM02B-SRSS-TB-LF-SN"
+			(at 115.57 238.76 0)
 			(effects
 				(font
@@
 			)
 		)
-		(property "Datasheet" "~"
-			(at 118.11 240.03 0)
+		(property "Datasheet" "https://lcsc.com/product-detail/Others_JST-Sales-America__JST-Sales-America-SM02B-SRSS-TB-LF-SN_C160402.html"
+			(at 113.03 238.76 0)
 			(effects
 				(font
@@
 			)
 		)
-		(property "Description" "Generic connector, single row, 01x02, script generated (kicad-library-utils/schlib/autogen/connector/)"
-			(at 118.11 240.03 0)
+		(property "Description" ""
+			(at 119.38 238.76 0)
 			(effects
 				(font
@@
 		)
 		(property "LCSC Part" "C160402"
-			(at 118.11 231.14 0)
+			(at 110.49 238.76 0)
 			(effects
 				(font
@@
 			)
 		)
+		(pin "4"
+		)
 		(pin "2"
 		)
 		(pin "1"
 		)
+		(pin "3"
+		)
 		(instances
 			(project ""
@@
 	)
 	(symbol
-		(lib_id "CM5_IO:ComputeModule5-CM5_GPIO")
+		(lib_id "New_Library:ComputeModule5-CM5_GPIO")
 		(at 119.38 134.62 0)
 		(unit 1)
@@
 			)
 		)
-		(property "Footprint" "CM5_MINIMA_local:Raspberry-Pi-5-Compute-Module_GPIO"
+		(property "Footprint" "CM5IO:Raspberry-Pi-5-Compute-Module_GPIO"
 			(at 118.364 140.462 0)
 			(effects
@@
 		(at 356.87 242.57 0)
 		(unit 1)
-		(exclude_from_sim yes)
+		(exclude_from_sim no)
 		(in_bom no)
-		(on_board yes)
+		(on_board no)
 		(dnp yes)
 		(fields_autoplaced yes)
 		(property "Reference" "M303"
-			(at 360.68 240.03 0)
+			(at 368.3 243.205 0)
 			(effects
 				(font
@@
 		)
 		(property "Value" "Compute-Module-4_H1.5mm"
-			(at 360.68 242.57 0)
+			(at 368.3 245.745 0)
 			(effects
 				(font
@@
 			)
 		)
-		(property "Footprint" "CM5_MINIMA_local:Compute-Module-4_H1.5mm"
-			(at 356.87 242.57 0)
+		(property "Footprint" "Antmicro-footprints:Compute-Module-4_H1.5mm"
+			(at 374.65 250.19 0)
 			(effects
 				(font
 					(size 1.27 1.27)
+					(thickness 0.15)
 				)
+				(justify left bottom)
 				(hide yes)
 			)
 		)
 		(property "Datasheet" "https://datasheets.raspberrypi.com/cm4/cm4-datasheet.pdf"
-			(at 356.87 242.57 0)
+			(at 374.65 252.73 0)
 			(effects
 				(font
 					(size 1.27 1.27)
+					(thickness 0.15)
 				)
+				(justify left bottom)
 				(hide yes)
 			)
 		)
-		(property "Description" "PCB Standoff, 1.5mm height, for Compute Module mounting"
+		(property "Description" ""
 			(at 356.87 242.57 0)
 			(effects
@@
 		)
 		(property "DNP" "DNP"
-			(at 360.68 245.1099 0)
+			(at 368.3 248.285 0)
 			(effects
 				(font
@@
 			)
 		)
-		(pin "1"
-		)
 		(instances

Commit message: with old version retraced and fixing
Parts:
- Module301: symbol New_Library:ComputeModule5-CM5_GPIO -> CM5_IO:ComputeModule5-CM5_GPIO
- Module302: symbol New_Library:ComputeModule5-CM5_HSS -> CM5_IO:ComputeModule5-CM5_HSS
Changed lines of the file:
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@@
 	)
 	(symbol
-		(lib_id "New_Library:ComputeModule5-CM5_HSS")
+		(lib_id "CM5_IO:ComputeModule5-CM5_HSS")
 		(at 298.45 135.89 0)
 		(unit 1)
@@
 	)
 	(symbol
-		(lib_id "New_Library:ComputeModule5-CM5_GPIO")
+		(lib_id "CM5_IO:ComputeModule5-CM5_GPIO")
 		(at 119.38 134.62 0)
 		(unit 1)
