File: CM5_MINIMA_REV3-main/IO.kicad_sch (KiCad schematic)
At the start: 19 parts, among them J502 I2C, J503 SPI, J601 JST_SHBM04B-SRSS-TB, SW501 TS-1010A-B, SW601 B3U-3100-P, U1 LIS3DH, U602 SN74LVC1G14DBVR

Commit message: warning fix - 17 left
Parts:
- D605, D606: footprint EasyEDA:LED-SMD_L1.7-W0.6-RD -> CM5_MINIMA_local:LED-SMD_L1.7-W0.6-RD
- SW501: footprint EasyEDA:SW-SMD_TS-1010A-B -> easyeda2kicad:SW-SMD_TS-1010A-B
- U602: symbol CM4IO:74LVC1G07_copy -> 74xGxx:74LVC1G07
Connections:
- no-connect marks 12 -> 13
Changed lines of the file:
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@@
 	)
 	(junction
-		(at 64.77 115.57)
-		(diameter 0)
-		(color 0 0 0 0)
-	)
-	(junction
 		(at 33.02 63.5)
 		(diameter 0)
@@
 	)
 	(no_connect
+		(at 67.31 45.72)
+	)
+	(no_connect
 		(at 115.57 62.23)
 	)
@@
 	(wire
 		(pts
-			(xy 66.04 35.56) (xy 68.58 35.56)
+			(xy 48.26 35.56) (xy 54.61 35.56)
 		)
 		(stroke
@@
 	(wire
 		(pts
-			(xy 76.2 33.02) (xy 76.2 22.86)
-		)
-		(stroke
-			(width 0)
-			(type solid)
-		)
-	)
-	(wire
-		(pts
 			(xy 33.02 59.69) (xy 33.02 63.5)
 		)
@@
 	(wire
 		(pts
-			(xy 64.77 115.57) (xy 67.31 115.57)
-		)
-		(stroke
-			(width 0)
-			(type default)
-		)
-	)
-	(wire
-		(pts
 			(xy 160.02 71.12) (xy 160.02 77.47)
 		)
@@
 	(wire
 		(pts
-			(xy 88.9 35.56) (xy 82.55 35.56)
-		)
-		(stroke
-			(width 0)
-			(type solid)
-		)
-	)
-	(wire
-		(pts
 			(xy 63.5 83.82) (xy 63.5 85.09)
 		)
@@
 	(wire
 		(pts
+			(xy 64.77 22.86) (xy 64.77 25.4)
+		)
+		(stroke
+			(width 0)
+			(type default)
+		)
+	)
+	(wire
+		(pts
 			(xy 34.29 101.6) (xy 34.29 125.73)
 		)
@@
 	(wire
 		(pts
+			(xy 82.55 35.56) (xy 88.9 35.56)
+		)
+		(stroke
+			(width 0)
+			(type default)
+		)
+	)
+	(wire
+		(pts
 			(xy 144.78 77.47) (xy 138.43 77.47)
 		)
@@
 	(wire
 		(pts
-			(xy 76.2 38.1) (xy 76.2 45.72)
+			(xy 186.69 82.55) (xy 186.69 86.36)
 		)
 		(stroke
@@
 	(wire
 		(pts
-			(xy 186.69 82.55) (xy 186.69 86.36)
+			(xy 177.8 31.75) (xy 176.53 31.75)
 		)
 		(stroke
@@
 	(wire
 		(pts
-			(xy 177.8 31.75) (xy 176.53 31.75)
+			(xy 161.29 80.01) (xy 167.64 80.01)
 		)
 		(stroke
@@
 	(wire
 		(pts
-			(xy 161.29 80.01) (xy 167.64 80.01)
+			(xy 144.78 77.47) (xy 144.78 82.55)
 		)
 		(stroke
@@
 	(wire
 		(pts
-			(xy 144.78 77.47) (xy 144.78 82.55)
+			(xy 64.77 45.72) (xy 64.77 49.53)
 		)
 		(stroke
@@
 	(hierarchical_label "nPWR_LED"
 		(shape input)
-		(at 66.04 35.56 180)
+		(at 48.26 35.56 180)
 		(effects
 			(font
@@
 			)
 		)
-		(property "Footprint" "EasyEDA:SW-SMD_TS-1010A-B"
+		(property "Footprint" "easyeda2kicad:SW-SMD_TS-1010A-B"
 			(at 39.37 115.57 0)
 			(effects
@@
 	(symbol
 		(lib_id "power:+5V")
-		(at 76.2 22.86 0)
+		(at 64.77 22.86 0)
 		(unit 1)
 		(exclude_from_sim no)
@@
 		(fields_autoplaced yes)
 		(property "Reference" "#PWR0516"
-			(at 76.2 26.67 0)
+			(at 64.77 26.67 0)
 			(effects
 				(font
@@
 		)
 		(property "Value" "+5V"
-			(at 76.2 17.78 0)
+			(at 64.77 17.78 0)
 			(effects
 				(font
@@
 		)
 		(property "Footprint" ""
-			(at 76.2 22.86 0)
+			(at 64.77 22.86 0)
 			(effects
 				(font
@@
 		)
 		(property "Datasheet" ""
-			(at 76.2 22.86 0)
+			(at 64.77 22.86 0)
 			(effects
 				(font
@@
 		)
 		(property "Description" "Power symbol creates a global label with name \"+5V\""
-			(at 76.2 22.86 0)
+			(at 64.77 22.86 0)
 			(effects
 				(font
@@
 	)
 	(symbol
+		(lib_name "R_Small_1")
 		(lib_id "Device:R_Small")
 		(at 152.4 68.58 0)
@@
 			)
 		)
-		(property "Datasheet" ""
+		(property "Datasheet" "~"
 			(at 152.4 68.58 0)
 			(effects
@@
 			)
 		)
-		(property "Description" ""
+		(property "Description" "Resistor, small symbol"
 			(at 152.4 68.58 0)
 			(effects
@@
 			)
 		)
-		(property "Datasheet" ""
+		(property "Datasheet" "~"
 			(at 160.02 68.58 0)
 			(effects
@@
 			)
 		)
-		(property "Description" ""
+		(property "Description" "Resistor, small symbol"
 			(at 160.02 68.58 0)
 			(effects
@@
 		(fields_autoplaced yes)
 		(property "Reference" "D606"
-			(at 142.24 23.1775 90)
+			(at 142.24 23.1774 90)
 			(effects
 				(font
@@
 		)
 		(property "Value" "GREEN"
-			(at 142.24 25.7175 90)
+			(at 142.24 25.7174 90)
 			(effects
 				(font
@@
 			)
 		)
-		(property "Footprint" "EasyEDA:LED-SMD_L1.7-W0.6-RD"
+		(property "Footprint" "CM5_MINIMA_local:LED-SMD_L1.7-W0.6-RD"
 			(at 138.43 22.86 0)
 			(effects
@@
 			)
 		)
-		(property "Datasheet" ""
+		(property "Datasheet" "~"
 			(at 138.43 22.86 0)
 			(effects
@@
 			)
 		)
-		(property "Description" ""
+		(property "Description" "Light emitting diode"
 			(at 138.43 22.86 0)
 			(effects
@@
 			)
 		)
+		(property "Sim.Pins" "1=K 2=A"
+			(at 138.43 22.86 0)
+			(effects
+				(font
+					(size 1.27 1.27)
+				)
+				(hide yes)
+			)
+		)
 		(pin "1"
 		)
@@
 	(symbol
 		(lib_id "power:GND")
-		(at 76.2 45.72 0)
+		(at 64.77 49.53 0)
 		(unit 1)
 		(exclude_from_sim no)
@@
 		(fields_autoplaced yes)
 		(property "Reference" "#PWR0607"
-			(at 76.2 52.07 0)
+			(at 64.77 55.88 0)
 			(effects
 				(font
@@
 		)
 		(property "Value" "GND"
-			(at 76.2 50.8 0)
+			(at 64.77 54.61 0)
 			(effects
 				(font
@@
 		)
 		(property "Footprint" ""
-			(at 76.2 45.72 0)
+			(at 64.77 49.53 0)
 			(effects
 				(font
@@
 		)
 		(property "Datasheet" ""
-			(at 76.2 45.72 0)
+			(at 64.77 49.53 0)
 			(effects
 				(font
@@
 		)
 		(property "Description" "Power symbol creates a global label with name \"GND\" , ground"
-			(at 76.2 45.72 0)
+			(at 64.77 49.53 0)
 			(effects
 				(font
@@
 	)
 	(symbol
-		(lib_name "74LVC1G07_copy_1")
-		(lib_id "CM4IO:74LVC1G07_copy")
-		(at 76.2 35.56 0)
+		(lib_id "74xGxx:74LVC1G07")
+		(at 69.85 35.56 0)
 		(unit 1)
 		(exclude_from_sim no)
@@
 		(dnp no)
 		(property "Reference" "U602"
-			(at 77.724 33.02 0)
+			(at 71.374 33.02 0)
 			(effects
 				(font
@@
 		)
 		(property "Value" "SN74LVC1G14DBVR"
-			(at 77.724 38.1 0)
+			(at 71.374 38.1 0)
 			(effects
 				(font
@@
 		)
 		(property "Footprint" "Package_TO_SOT_SMD:SOT-353_SC-70-5"
-			(at 76.2 35.56 0)
+			(at 69.85 35.56 0)
 			(effects
 				(font
@@
 			)
 		)
-		(property "Datasheet" "https://www.lcsc.com/datasheet/lcsc_datasheet_2405141143_UMW-Youtai-Semiconductor-Co---Ltd--SN74LVC1G14DBVR_C434069.pdf"
-			(at 76.2 35.56 0)
+		(property "Datasheet" "https://www.ti.com/lit/ds/symlink/sn74lvc1g07.pdf"
+			(at 69.85 35.56 0)
 			(effects
 				(font
@@
 			)
 		)
-		(property "Description" ""
-			(at 76.2 35.56 0)
+		(property "Description" "Single Buffer Gate, Open Drain, Low-Voltage CMOS"
+			(at 69.85 35.56 0)
 			(effects
 				(font
@@
 		)
 		(property "Part Description" "Buffer, Non-Inverting 1 Element 1 Bit per Element Open Drain Output SOT-353"
-			(at 76.2 35.56 0)
+			(at 69.85 35.56 0)
 			(effects
 				(font
@@
 		)
 		(property "P/N" "SN74LVC1G14DBVR"
-			(at 76.2 35.56 0)
+			(at 69.85 35.56 0)
 			(effects
 				(font
@@
 	)
 	(symbol
+		(lib_name "LED_1")
 		(lib_id "Device:LED")
 		(at 88.9 22.86 90)
@@
 		(fields_autoplaced yes)
 		(property "Reference" "D605"
-			(at 92.71 23.1775 90)
+			(at 92.71 23.1774 90)
 			(effects
 				(font
@@
 		)
 		(property "Value" "GREEN"
-			(at 92.71 25.7175 90)
+			(at 92.71 25.7174 90)
 			(effects
 				(font
@@
 			)
 		)
-		(property "Footprint" "EasyEDA:LED-SMD_L1.7-W0.6-RD"
+		(property "Footprint" "CM5_MINIMA_local:LED-SMD_L1.7-W0.6-RD"
 			(at 88.9 22.86 0)
 			(effects
@@
 			)
 		)
-		(property "Datasheet" ""
+		(property "Datasheet" "~"
 			(at 88.9 22.86 0)
 			(effects
@@
 			)
 		)
-		(property "Description" ""
+		(property "Description" "Light emitting diode"
 			(at 88.9 22.86 0)
 			(effects
@@
 			(at 88.9 22.86 0)
 			(effects
+				(font
+					(size 1.27 1.27)
+				)
+				(hide yes)
+			)
+		)
+		(property "Sim.Pins" "1=K 2=A"
+			(at 88.9 22.86 0)
+			(effects

Commit message: warning fix - 0  in schematic
Parts:
- SW501: footprint easyeda2kicad:SW-SMD_TS-1010A-B -> CM5_MINIMA_local:SW-SMD_TS-1010A-B
Changed lines of the file:
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@@
 			)
 		)
-		(property "Footprint" "easyeda2kicad:SW-SMD_TS-1010A-B"
+		(property "Footprint" "CM5_MINIMA_local:SW-SMD_TS-1010A-B"
 			(at 39.37 115.57 0)
 			(effects
