File: CM5_MINIMA_REV3-main/DSI_CSI.kicad_sch (KiCad schematic)
At the start: 1 part, among them J802 Conn_01x22_Female

Commit message: warning fix - 17 left
Parts:
- J802: footprint CM5IO:Hirose_FH12-22S-0.5SH_1x22-1MP_P0.50mm_Horizontal -> CM5_MINIMA_local:Hirose_FH12-22S-0.5SH_1x22-1MP_P0.50mm_Horizontal
Changed lines of the file:
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@@
 			)
 		)
-		(property "Footprint" "CM5IO:Hirose_FH12-22S-0.5SH_1x22-1MP_P0.50mm_Horizontal"
+		(property "Footprint" "CM5_MINIMA_local:Hirose_FH12-22S-0.5SH_1x22-1MP_P0.50mm_Horizontal"
 			(at 111.76 59.69 0)
 			(effects

Commit message: Revert CM5_MINIMA_REV3-main to pre-warning-fix state (feae2c2) - fix component mismatches
Parts:
- J802: footprint CM5_MINIMA_local:Hirose_FH12-22S-0.5SH_1x22-1MP_P0.50mm_Horizontal -> CM5IO:Hirose_FH12-22S-0.5SH_1x22-1MP_P0.50mm_Horizontal
Changed lines of the file:
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@@
 			)
 		)
-		(property "Footprint" "CM5_MINIMA_local:Hirose_FH12-22S-0.5SH_1x22-1MP_P0.50mm_Horizontal"
+		(property "Footprint" "CM5IO:Hirose_FH12-22S-0.5SH_1x22-1MP_P0.50mm_Horizontal"
 			(at 111.76 59.69 0)
 			(effects
