File: CM5_MINIMA_REV3-main/USB.kicad_sch (KiCad schematic)
At the start: 9 parts, among them U701 AP22653W6

Commit message: with old version retraced and fixing
Parts:
- USB701: footprint EasyEDA:USB-C-SMD_TYPEC-305-ACP16H458 -> easyeda2kicad:USB-C-SMD_TYPEC-305-ACP16H458
Changed lines of the file:
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@@
 			)
 		)
-		(property "Footprint" "EasyEDA:USB-C-SMD_TYPEC-305-ACP16H458"
+		(property "Footprint" "easyeda2kicad:USB-C-SMD_TYPEC-305-ACP16H458"
 			(at 50.8 110.49 0)
 			(effects
