File: CM5_MINIMA_REV3-main/Ethernet.kicad_sch (KiCad schematic)
At the start: 7 parts, among them J1 GLPLX-SMT-188S7, U401 TPD4EUSB30, U402 TPD4EUSB30

Commit message: with old version retraced and fixing
Parts:
- U401, U402: symbol CM4IO:TPD4EUSB30 -> CM5IO:TPD4EUSB30
Changed lines of the file:
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@@
+	)
+	(junction
+		(at 146.05 76.2)
+		(diameter 0)
+		(color 0 0 0 0)
 	)
 	(junction
@@
 	)
 	(junction
-		(at 146.05 76.2)
-		(diameter 0)
-		(color 0 0 0 0)
-	)
-	(junction
 		(at 118.11 60.96)
 		(diameter 0)
@@
 	(wire
 		(pts
+			(xy 146.05 73.66) (xy 146.05 76.2)
+		)
+		(stroke
+			(width 0)
+			(type default)
+		)
+	)
+	(wire
+		(pts
+			(xy 146.05 76.2) (xy 146.05 78.74)
+		)
+		(stroke
+			(width 0)
+			(type default)
+		)
+	)
+	(wire
+		(pts
 			(xy 135.89 85.09) (xy 135.89 87.63)
 		)
@@
 	(wire
 		(pts
-			(xy 146.05 78.74) (xy 146.05 76.2)
-		)
-		(stroke
-			(width 0)
-			(type default)
-		)
-	)
-	(wire
-		(pts
 			(xy 185.42 67.31) (xy 185.42 52.07)
 		)
@@
 		(pts
 			(xy 179.07 54.61) (xy 189.23 54.61)
-		)
-		(stroke
-			(width 0)
-			(type default)
-		)
-	)
-	(wire
-		(pts
-			(xy 146.05 73.66) (xy 146.05 76.2)
 		)
 		(stroke
@@
 	)
 	(symbol
-		(lib_id "CM4IO:TPD4EUSB30")
+		(lib_id "CM5IO:TPD4EUSB30")
 		(at 100.33 81.28 0)
 		(unit 1)
@@
 			)
 		)
-		(property "Datasheet" ""
+		(property "Datasheet" "http://www.ti.com/lit/ds/symlink/tpd2eusb30a.pdf"
 			(at 100.33 81.28 0)
 			(effects
@@
 			)
 		)
-		(property "Description" ""
+		(property "Description" "4-Channel ESD Protection for Super-Speed USB 3.0 Interface, USON-10"
 			(at 100.33 81.28 0)
 			(effects
@@
 	)
 	(symbol
-		(lib_id "CM4IO:TPD4EUSB30")
+		(lib_id "CM5IO:TPD4EUSB30")
 		(at 59.69 81.28 0)
 		(unit 1)
@@
 			)
 		)
-		(property "Datasheet" ""
+		(property "Datasheet" "http://www.ti.com/lit/ds/symlink/tpd2eusb30a.pdf"
 			(at 59.69 81.28 0)
 			(effects
@@
 			)
 		)
-		(property "Description" ""
+		(property "Description" "4-Channel ESD Protection for Super-Speed USB 3.0 Interface, USON-10"
 			(at 59.69 81.28 0)
 			(effects
