File: RelaySwitch/RelaySwitch_C6 - Copy/RelaySwitch_C6.kicad_sch (KiCad schematic)
At the start: 39 parts, among them J1 AC_MAINS_IN, J3 LOAD_CH1, J4 LOAD_CH2, J5 SW1_INPUT, J6 SW2_INPUT, K1 G5Q-1-DC5, K2 G5Q-1-DC5, Q1 MMBT8050, Q2 MMBT8050, U1 HLK-2M05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

Commit message: For review
Parts:
- removed R10: 1m, Resistor_SMD:R_2512_6332Metric, symbol Device:R
- added C2: 10u, Capacitor_SMD:C_0402_1005Metric, symbol Device:C_Small
- added C3: 100n, Capacitor_SMD:C_0402_1005Metric, symbol Device:C_Small
- J1: footprint TerminalBlock_Degson:TerminalBlock_Degson_DG250-3.5-03P_1x03_P3.50mm_45Degree -> seeed esp32:CONN-TH_3P-P5.00_WJ128V-5.0-3P; symbol Connector:Screw_Terminal_01x03 -> WJ128V3P:WJ128V-5.0-3P; Check_prices (none) -> https://www.snapeda.com/parts/TB0011-350-03BE/Same+Sky/view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; Description_1 (none) -> 3 Position Wire to Board Terminal Block Horizontal with Boa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; DigiKey_Part_Number (none) -> 2223-TB0011-350-03BE-ND; LCSC Part (none) -> C8270; MANUFACTURER (none) -> SAMESKY; MF (none) -> Same Sky; MP (none) -> TB0011-350-03BE; Package (none) -> None; SnapEDA_Link (none) -> https://www.snapeda.com/parts/TB0011-350-03BE/Same+Sky/view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
- J3, J4, J5, J6: footprint TerminalBlock_Degson:TerminalBlock_Degson_DG250-3.5-02P_1x02_P3.50mm_45Degree -> seeed esp32:CONN-TH_2P-P5.00_WJ128V-5.0-2P; symbol Connector:Screw_Terminal_01x02 -> WJ128V:WJ128V-5.0-2P; CREATOR (none) -> ASHISH; Check_prices (none) -> https://www.snapeda.com/parts/TB0011-350-02BE/Same+Sky/view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; Description_1 (none) -> 2 Position Wire to Board Terminal Block Horizontal with Boa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; DigiKey_Part_Number (none) -> 2223-TB0011-350-02BE-ND; LCSC Part (none) -> C8269; MANUFACTURER (none) -> Same Sky; MAXIMUM_PACKAGE_HEIGHT (none) -> 8.5mm; MF (none) -> Same Sky; MP (none) -> TB0011-350-02BE; PARTREV (none) -> 1.0; Package (none) -> None; STANDARD (none) -> Manufacturer Recommendations; SnapEDA_Link (none) -> https://www.snapeda.com/parts/TB0011-350-02BE/Same+Sky/view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
- R18: footprint Resistor_SMD:R_Shunt_Vishay_WSK2512_6332Metric_T2.66mm -> XIAO_Series_Footprints:RES_WSK2512R0100FEA; symbol Device:R -> WSK2512R0100FEA:WSK2512R0100FEA; Check_prices (none) -> https://www.snapeda.com/parts/WSK2512R0100FEA/Vishay/view-p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; Description_1 (none) -> Metal Strip Low Ohmic Smnt Resistor 2512 Case 10mOhm +/-1% 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; DigiKey_Part_Number (none) -> 541-WSK2512R0100FEACT-ND; MANUFACTURER (none) -> Vishay Dale; MAXIMUM_PACKAGE_HEIGHT (none) -> 0.889mm; MF (none) -> Vishay; MP (none) -> WSK2512R0100FEA; PARTREV (none) -> 04-Apr-2022; Package (none) -> None; SNAPEDA_PN (none) -> WSK2512R0100FEA; STANDARD (none) -> Manufacturer Recommendations; SnapEDA_Link (none) -> https://www.snapeda.com/parts/WSK2512R0100FEA/Vishay/view-p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
- U2: footprint XIAO_Series_Footprints:XIAO-ESP32-C6-SMD -> XIAO_Series_Footprints:XIAO-ESP32-C6-DIP
- U5: footprint HLW8012:SOIC8 -> seeed esp32:SOIC8
Connections:
- net +3V3: now also C3.1; no longer C5.1
- net +5V: now also C5.1, C2.1
- net GND: now also U5.4 (V2P), C2.2, C3.2; no longer U5.3 (V1N)
- net L: now also R18.I1; no longer R18.1, U5.4 (V2P)
- net L_Sense: now also R18.I2; no longer R18.2
- net at R13.2, R9.1, U5.2 (V1P): now also R18.E1
- new net: R18.E2, U5.3 (V1N)
Other:
- moved on the sheet: C5, C6
